File: mechanical_hardware/schematics/schematics.kicad_sch (KiCad schematic)
At the start: 19 parts, among them J1 Raspberry_Pi_4, J4 TB6612FNG, J5 Encoder, J6 Encoder, M1 Motor_DC, M2 Motor_DC, SW2 SW_DIP_x02, U1 5.1V, U2 5V, U3 11.5V, U4 ESP32-DevKitC, U5 MPU-9250, U6 MPU-6050

Commit message: changed wiring, accidentally wired encoder with boot pin which caused problems
Connections:
- net at J5.E-A (Pin_5): now also U4.5 (VDET_1/GPIO34/ADC1_CH6); no longer U4.25 (GPIO0/BOOT/ADC2_CH1)
- net at U4.23 (MTDO/GPIO15/ADC2_CH3): no longer J6.E-A (Pin_5)
- net at U4.24 (ADC2_CH2/GPIO2): no longer J6.E-B (Pin_3)
- net at U4.3 (SENSOR_VP/GPIO36/ADC1_CH0): now also J6.E-A (Pin_5)
- net at U4.6 (VDET_2/GPIO35/ADC1_CH7): now also J6.E-B (Pin_3)
Changed lines of the file:
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@@
+	(wire
+		(pts
+			(xy 254 134.62) (xy 158.75 134.62)
+		)
+		(stroke
+			(width 0)
+			(type default)
+		)
+	)
 	(wire
 		(pts
@@
 	(wire
 		(pts
+			(xy 166.37 173.99) (xy 170.18 173.99)
+		)
+		(stroke
+			(width 0)
+			(type default)
+		)
+	)
+	(wire
+		(pts
 			(xy 245.11 168.91) (xy 236.22 168.91)
 		)
@@
 	(wire
 		(pts
-			(xy 156.21 166.37) (xy 170.18 166.37)
+			(xy 166.37 215.9) (xy 166.37 173.99)
 		)
 		(stroke
@@
 	(wire
 		(pts
-			(xy 156.21 218.44) (xy 156.21 166.37)
+			(xy 156.21 218.44) (xy 156.21 176.53)
 		)
 		(stroke
@@
 	(wire
 		(pts
+			(xy 158.75 134.62) (xy 158.75 171.45)
+		)
+		(stroke
+			(width 0)
+			(type default)
+		)
+	)
+	(wire
+		(pts
 			(xy 312.42 175.26) (xy 261.62 175.26)
 		)
@@
 	(wire
 		(pts
-			(xy 236.22 156.21) (xy 251.46 156.21)
-		)
-		(stroke
-			(width 0)
-			(type default)
-		)
-	)
-	(wire
-		(pts
 			(xy 280.67 152.4) (xy 280.67 165.1)
 		)
@@
 	(wire
 		(pts
+			(xy 254 153.67) (xy 254 134.62)
+		)
+		(stroke
+			(width 0)
+			(type default)
+		)
+	)
+	(wire
+		(pts
 			(xy 255.27 259.08) (xy 264.16 259.08)
 		)
@@
 	(wire
 		(pts
-			(xy 251.46 179.07) (xy 251.46 156.21)
-		)
-		(stroke
-			(width 0)
-			(type default)
-		)
-	)
-	(wire
-		(pts
 			(xy 203.2 123.19) (xy 274.32 123.19)
 		)
@@
 	(wire
 		(pts
+			(xy 251.46 179.07) (xy 251.46 215.9)
+		)
+		(stroke
+			(width 0)
+			(type default)
+		)
+	)
+	(wire
+		(pts
 			(xy 167.64 223.52) (xy 203.2 223.52)
 		)
@@
 	(wire
 		(pts
+			(xy 158.75 171.45) (xy 170.18 171.45)
+		)
+		(stroke
+			(width 0)
+			(type default)
+		)
+	)
+	(wire
+		(pts
 			(xy 369.57 163.83) (xy 369.57 190.5)
 		)
@@
 	(wire
 		(pts
+			(xy 254 153.67) (xy 318.77 153.67)
+		)
+		(stroke
+			(width 0)
+			(type default)
+		)
+	)
+	(wire
+		(pts
 			(xy 152.4 123.19) (xy 46.99 123.19)
 		)
@@
 	(wire
 		(pts
+			(xy 251.46 215.9) (xy 166.37 215.9)
+		)
+		(stroke
+			(width 0)
+			(type default)
+		)
+	)
+	(wire
+		(pts
 			(xy 261.62 137.16) (xy 205.74 137.16)
 		)
@@
 	(wire
 		(pts
+			(xy 156.21 176.53) (xy 170.18 176.53)
+		)
+		(stroke
+			(width 0)
+			(type default)
+		)
+	)
+	(wire
+		(pts
 			(xy 171.45 76.2) (xy 160.02 76.2)
 		)
@@
 		)
 		(stroke
-			(width 0)
-			(type default)
-		)
-	)
-	(wire
-		(pts
-			(xy 236.22 153.67) (xy 318.77 153.67)
-		)
-		(stroke
